File: PCB/dapt/dapt.kicad_pcb (KiCad board)
At the start: 2 copper layers, 62.5 x 109 mm, 42 parts

Commit message: a
Parts:
- USB12, USB23: moved to B.Cu
- moved USB23 15.7 mm to (88.3, 71.4), turned to 180 degrees
- moved USB22 9.66 mm to (88.1, 86.2), turned to 180 degrees
- moved R22 4.75 mm to (88.3, 79.0), turned to 180 degrees
- moved USB12 4.41 mm to (74.2, 71.3), turned to 180 degrees
- moved R21 1.25 mm to (88.3, 82.0), turned to 180 degrees
Routing:
- net /C_female_C_female/VBUS: track 0.00 -> 30.0 mm, vias 0 -> 2
- net /A_female_C_male1/VBUS: track 0.00 -> 24.9 mm, vias 0 -> 3
- net /A_female_C_male1/D-: track 0.00 -> 24.5 mm
- net /A_female_C_male3/D-: track 0.00 -> 24.0 mm
- net /A_female_C_male/D-: track 0.00 -> 23.9 mm
- net /A_female_C_male2/D-: track 0.00 -> 22.2 mm
- net /C_female_C_female/D-: track 0.00 -> 21.1 mm
- net /C_female_C_female/D+: track 0.00 -> 20.8 mm
- net /A_female_C_male1/D+: track 0.00 -> 20.5 mm
- net /A_female_C_male/D+: track 0.00 -> 20.1 mm
- net /A_female_C_male3/D+: track 0.00 -> 19.4 mm
- net /C_female_micro_male/GND: track 0.00 -> 19.1 mm
- net /C_female_micro_male/D+: track 0.00 -> 18.6 mm
- net /C_female_micro_male1/D+: track 0.00 -> 18.6 mm
- net /A_female_C_male3/VBUS: track 0.00 -> 18.5 mm, vias 0 -> 2
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- added copper zone on F.Cu, net /A_female_A_female/GND
- added copper zone on B.Cu, net /A_female_A_female/VBUS
- added copper zone on F.Cu, net /A_female_C_male/GND
- added copper zone on B.Cu, net /A_female_C_male/VBUS
- added copper zone on F.Cu, net /A_female_C_male1/GND
- added copper zone on B.Cu, net /A_female_C_male1/VBUS
- added copper zone on F.Cu, net /A_female_C_male2/GND
- added copper zone on B.Cu, net /A_female_C_male2/VBUS
- added copper zone on F.Cu, net /A_female_C_male3/GND
- added copper zone on B.Cu, net /A_female_C_male3/VBUS
- added copper zone on F.Cu, net /A_male_A_male/GND
- added copper zone on B.Cu, net /A_male_A_male/VBUS
- added copper zone on F.Cu, net /A_male_C_female/GND
- added copper zone on B.Cu, net /A_male_C_female/VBUS
- added copper zone on F.Cu, net /A_male_C_female1/GND
- added copper zone on B.Cu, net /A_male_C_female1/VBUS
- added copper zone on F.Cu, net /C_female_C_female/GND
- added copper zone on B.Cu, net /C_female_C_female/VBUS
- added copper zone on F.Cu, net /C_female_micro_male/GND
- added copper zone on B.Cu, net /C_female_micro_male/VBUS
- added copper zone on F.Cu, net /C_female_micro_male1/GND
- added copper zone on B.Cu, net /C_female_micro_male1/VBUS
Other:
- board size 62.5 x 109 mm -> 64 x 109.5 mm

Commit message: I hate panelization
Parts:
- added B1: MouseBite, Panelization:MouseBite-Slot_2.0x2.0mm_inset_D0.5mm_P0.85mm_5h, F.Cu at (80.5, 139.0)
- added B11: MouseBite, Panelization:MouseBite-Slot_2.0x2.0mm_inset_D0.5mm_P0.85mm_5h, F.Cu at (46.5, 140.2)
- added B12: MouseBite, Panelization:MouseBite-Slot_2.0x2.0mm_inset_D0.5mm_P0.85mm_5h, F.Cu at (80.0, 119.0)
- added B13: MouseBite, Panelization:MouseBite-Slot_2.0x2.0mm_inset_D0.5mm_P0.85mm_5h, F.Cu at (57.0, 111.8)
- added B2: MouseBite, Panelization:MouseBite-Slot_2.0x2.0mm_inset_D0.5mm_P0.85mm_5h, F.Cu at (56.7, 149.3)
- added B4: MouseBite, Panelization:MouseBite-Slot_2.0x2.0mm_inset_D0.5mm_P0.85mm_5h, F.Cu at (71.6, 128.3)
- added B6: MouseBite, Panelization:MouseBite-Slot_2.0x2.0mm_inset_D0.5mm_P0.85mm_5h, F.Cu at (73.2, 148.7)
- added B7: MouseBite, Panelization:MouseBite-Slot_2.0x2.0mm_inset_D0.5mm_P0.85mm_5h, F.Cu at (73.1, 109.2)
- added B7: MouseBite, Panelization:MouseBite-Slot_2.0x2.0mm_inset_D0.5mm_P0.85mm_5h, F.Cu at (48.3, 118.6)
- added B7: MouseBite, Panelization:MouseBite-Slot_2.0x2.0mm_inset_D0.5mm_P0.85mm_5h, F.Cu at (58.2, 128.3)
- moved USB15 8.73 mm to (51.0, 110.1)
- moved USB25 8.73 mm to (46.6, 110.1)
- moved R10 6.20 mm to (48.2, 127.7)
- moved R9 6.20 mm to (51.2, 127.7)
- moved USB10 6.20 mm to (43.9, 128.9)
- moved USB20 5.99 mm to (52.7, 148.7)
- moved R19 5.99 mm to (49.7, 149.2)
- moved R20 5.99 mm to (46.7, 149.2)
- moved USB21 5.99 mm to (42.4, 148.7)
- moved USB16 5.54 mm to (77.0, 108.0)
- moved USB17 5.54 mm to (82.5, 108.0)
- moved USB8 4.87 mm to (52.8, 127.0)
- moved R7 4.07 mm to (83.8, 148.5)
- moved R8 4.07 mm to (80.8, 148.5)
- moved USB7 4.07 mm to (86.7, 148.0)
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Routing:
- net /A_female_C_male1/VBUS: track 24.9 -> 0.00 mm, vias 3 -> 0
- net /A_female_C_male1/GND: track 15.2 -> 32.8 mm, vias 2 -> 4
- net /A_female_C_male1/D-: track 24.5 -> 28.6 mm
- net Net-(USB8-CC1): track 9.77 -> 13.0 mm, vias 1 -> 2
Other:
- board size 64 x 109.5 mm -> 60.2 x 109.5 mm
