File: PCB/dapt/dapt.kicad_sch (KiCad schematic)
At the start: 0 parts

Commit message: I hate panelization
Parts:
- added B1, B10, B11, B12, B13, B2, B3, B4, B5, B6, B7, B8, B9: MouseBite, Panelization:MouseBite-Slot_2.0x2.0mm_inset_D0.5mm_P0.85mm_5h, symbol Mechanical:MouseBite
